File: PowerAdjustmentMonitor.sch (KiCad schematic (older format))
At the start: 0 parts

Commit message: M3 U6
Power Control, Conditioning and Monitoring module
Parts:
- added JP? (x3): JUMPER, ~, symbol JUMPER
- added R? (x8): R, ~, symbol R
- added R? (x2): RVAR, ~, symbol RVAR
- added U? (x2): LM317, ~, symbol LM317
- added U? (x2): 7805, ~, symbol 7805
- added U? (x2): LM324, ~, symbol LM324
Connections:
- net labels added: +12V, +3.3V, +5V, -12V, 3V3_MON, 5V_MON, AGND, FE_V+, FE_V-, GND, V+_ADJ, V+_ADJ_MON, V+_CURR_MON, V+_MON, V-_ADJ, V-_ADJ_MON, V-_CURR_MON, V-_MON
- wire segments 0 -> 79
