File: Thermocouple.sch (KiCad schematic (older format))
At the start: 0 parts

Commit message: Module 2.Unit 15
Defining you inputs and outputs
Changed lines of the file:
@@
 Text HLabel 8150 2300 2    60   Input ~ 0
 TC IN -
+Text HLabel 2550 2050 0    60   Input ~ 0
+MOSI
+Text HLabel 2550 2300 0    60   Output ~ 0
+MISO
+Text HLabel 2550 2600 0    60   Input ~ 0
+SCLK
+Text HLabel 2550 2900 0    60   Input ~ 0
+CS_N
 $EndSCHEMATC

Commit message: Module 3.Unit 1
Parts:
- added C?: C, ~, symbol C
- added D?: ZENER, ~, symbol ZENER
- added R? (x7): R, ~, symbol R
- added U? (x4): LM324, ~, symbol LM324
- added U? (x2): MCP3553-E/SN, SO8, symbol MCP3553-E/SN
Connections:
- net CS_N: now also U?.7 (~CS~)
- net MISO: now also U?.6 (SDO/~RDY~)
- net SCLK: now also U?.5 (SCK)
- net TC IN +: now also U?.3 (+)
- net TC IN -: now also U?.3 (+)
- new net: R?.1, R?.2, U?.1
- new net: R?.1, R?.2, U?.2 (-) (x3)
- new net: R?.2, R?.2, U?.1
- new net: R?.1, U?.1, U?.2 (Vin+)
- new net: R?.1, R?.2, U?.3 (+)
- new net: U?.1, U?.2 (-), U?.2 (Vin+)
- new net +12V: D?.2 (K), U?.3 (+), U?.4 (V+), U?.4 (V+), U?.4 (V+)
- new net -12V: U?.11 (V-), U?.11 (V-), U?.11 (V-)
- new net AGND: D?.1 (A), R?.1, U?.3 (Vin-), U?.3 (Vin-)
Other:
- note added: "16-24 Bit ADC"
- note added: "Analog/TC Control"
- note added: "General Temp Sensor"
- note added: "Intermediate Amp"
